Commit message: Set effort to -1 to fix no control in gazebo

File: robot_specific_config/abb_irb4600_support/urdf/irb4600_20_250_macro.xacro (robot description, xacro)
@@ -109,5 +109,5 @@
       <parent link="${prefix}base_link"/>
       <child link="${prefix}link_1"/>
-      <limit effort="0" lower="${radians(-180)}" upper="${radians(180)}" velocity="${radians(175)}"/>
+      <limit effort="-1" lower="${radians(-180)}" upper="${radians(180)}" velocity="${radians(175)}"/>
     </joint>
     <joint type="revolute" name="${prefix}joint_2">
@@ -116,5 +116,5 @@
       <parent link="${prefix}link_1"/>
       <child link="${prefix}link_2"/>
-      <limit effort="0" lower="${radians(-90)}" upper="${radians(150)}" velocity="${radians(175)}"/>
+      <limit effort="-1" lower="${radians(-90)}" upper="${radians(150)}" velocity="${radians(175)}"/>
     </joint>
     <joint type="revolute" name="${prefix}joint_3">
@@ -123,5 +123,5 @@
       <parent link="${prefix}link_2"/>
       <child link="${prefix}link_3"/>
-      <limit effort="0" lower="${radians(-180)}" upper="${radians(75)}" velocity="${radians(175)}"/>
+      <limit effort="-1" lower="${radians(-180)}" upper="${radians(75)}" velocity="${radians(175)}"/>
     </joint>
     <joint type="revolute" name="${prefix}joint_4">
@@ -130,5 +130,5 @@
       <parent link="${prefix}link_3"/>
       <child link="${prefix}link_4"/>
-      <limit effort="0" lower="${radians(-400)}" upper="${radians(400)}" velocity="${radians(360)}"/>
+      <limit effort="-1" lower="${radians(-400)}" upper="${radians(400)}" velocity="${radians(360)}"/>
     </joint>
     <joint type="revolute" name="${prefix}joint_5">
@@ -137,5 +137,5 @@
       <parent link="${prefix}link_4"/>
       <child link="${prefix}link_5"/>
-      <limit effort="0" lower="${radians(-125)}" upper="${radians(120)}" velocity="${radians(360)}"/>
+      <limit effort="-1" lower="${radians(-125)}" upper="${radians(120)}" velocity="${radians(360)}"/>
     </joint>
     <joint type="revolute" name="${prefix}joint_6">
@@ -144,5 +144,5 @@
       <parent link="${prefix}link_5"/>
       <child link="${prefix}link_6"/>
-      <limit effort="0" lower="${radians(-400)}" upper="${radians(400)}" velocity="${radians(500)}"/>
+      <limit effort="-1" lower="${radians(-400)}" upper="${radians(400)}" velocity="${radians(500)}"/>
     </joint>
     <!-- end of joint list -->

File: robot_specific_config/abb_irb4600_support/urdf/irb4600_40_255_macro.xacro (robot description, xacro)
@@ -131,5 +131,5 @@
       <parent link="${prefix}base_link"/>
       <child link="${prefix}link_1"/>
-      <limit effort="0" lower="${radians(-180)}" upper="${radians(180)}" velocity="${radians(175)}"/>
+      <limit effort="-1" lower="${radians(-180)}" upper="${radians(180)}" velocity="${radians(175)}"/>
     </joint>
     <joint type="revolute" name="${prefix}joint_2">
@@ -138,5 +138,5 @@
       <parent link="${prefix}link_1"/>
       <child link="${prefix}link_2"/>
-      <limit effort="0" lower="${radians(-90)}" upper="${radians(150)}" velocity="${radians(175)}"/>
+      <limit effort="-1" lower="${radians(-90)}" upper="${radians(150)}" velocity="${radians(175)}"/>
     </joint>
     <joint type="revolute" name="${prefix}joint_3">
@@ -145,5 +145,5 @@
       <parent link="${prefix}link_2"/>
       <child link="${prefix}link_3"/>
-      <limit effort="0" lower="${radians(-180)}" upper="${radians(75)}" velocity="${radians(175)}"/>
+      <limit effort="-1" lower="${radians(-180)}" upper="${radians(75)}" velocity="${radians(175)}"/>
     </joint>
     <joint type="revolute" name="${prefix}joint_4">
@@ -152,5 +152,5 @@
       <parent link="${prefix}link_3"/>
       <child link="${prefix}link_4"/>
-      <limit effort="0" lower="${radians(-400)}" upper="${radians(400)}" velocity="${radians(250)}"/>
+      <limit effort="-1" lower="${radians(-400)}" upper="${radians(400)}" velocity="${radians(250)}"/>
     </joint>
     <joint type="revolute" name="${prefix}joint_5">
@@ -159,5 +159,5 @@
       <parent link="${prefix}link_4"/>
       <child link="${prefix}link_5"/>
-      <limit effort="0" lower="${radians(-125)}" upper="${radians(120)}" velocity="${radians(250)}"/>
+      <limit effort="-1" lower="${radians(-125)}" upper="${radians(120)}" velocity="${radians(250)}"/>
     </joint>
     <joint type="revolute" name="${prefix}joint_6">
@@ -166,5 +166,5 @@
       <parent link="${prefix}link_5"/>
       <child link="${prefix}link_6"/>
-      <limit effort="0" lower="${radians(-400)}" upper="${radians(400)}" velocity="${radians(360)}"/>
+      <limit effort="-1" lower="${radians(-400)}" upper="${radians(400)}" velocity="${radians(360)}"/>
     </joint>
     <!-- end of joint list -->

File: robot_specific_config/abb_irb4600_support/urdf/irb4600_60_205_macro.xacro (robot description, xacro)
@@ -109,5 +109,5 @@
       <parent link="${prefix}base_link"/>
       <child link="${prefix}link_1"/>
-      <limit effort="0" lower="-3.141" upper="3.141" velocity="3.054"/>
+      <limit effort="-1" lower="-3.141" upper="3.141" velocity="3.054"/>
     </joint>
     <joint type="revolute" name="${prefix}joint_2">
@@ -116,5 +116,5 @@
       <parent link="${prefix}link_1"/>
       <child link="${prefix}link_2"/>
-      <limit effort="0" lower="-1.570" upper="2.617" velocity="3.054"/>
+      <limit effort="-1" lower="-1.570" upper="2.617" velocity="3.054"/>
     </joint>
     <joint type="revolute" name="${prefix}joint_3">
@@ -123,5 +123,5 @@
       <parent link="${prefix}link_2"/>
       <child link="${prefix}link_3"/>
-      <limit effort="0" lower="-3.141" upper="1.308" velocity="3.054"/>
+      <limit effort="-1" lower="-3.141" upper="1.308" velocity="3.054"/>
     </joint>
     <joint type="revolute" name="${prefix}joint_4">
@@ -130,5 +130,5 @@
       <parent link="${prefix}link_3"/>
       <child link="${prefix}link_4"/>
-      <limit effort="0" lower="-6.981" upper="6.981" velocity="4.363"/>
+      <limit effort="-1" lower="-6.981" upper="6.981" velocity="4.363"/>
     </joint>
     <joint type="revolute" name="${prefix}joint_5">
@@ -137,5 +137,5 @@
       <parent link="${prefix}link_4"/>
       <child link="${prefix}link_5"/>
-      <limit effort="0" lower="-2.181" upper="2.094" velocity="4.363"/>
+      <limit effort="-1" lower="-2.181" upper="2.094" velocity="4.363"/>
     </joint>
     <joint type="revolute" name="${prefix}joint_6">
@@ -144,5 +144,5 @@
       <parent link="${prefix}link_5"/>
       <child link="${prefix}link_6"/>
-      <limit effort="0" lower="-6.981" upper="6.981" velocity="6.283"/>
+      <limit effort="-1" lower="-6.981" upper="6.981" velocity="6.283"/>
     </joint>
     <!-- end of joint list -->
