Commit message: add inertial values to irb4600

File: robot_specific_config/abb_irb4600_support/urdf/irb4600_40_255_macro.xacro (robot description, xacro)
@@ -3,4 +3,5 @@
   <xacro:macro name="abb_irb4600_40_255" params="prefix">
     <xacro:include filename="$(find abb_resources)/urdf/common_materials.xacro"/>
+    <xacro:include filename="$(find abb_irb4600_support)/urdf/irb4600.inertial_macro.xacro"/>
     <!-- link list -->
     <link name="${prefix}base_link">
@@ -17,4 +18,7 @@
         <xacro:material_abb_graphite_white/>
       </visual>
+      <xacro:cylinder_inertial radius="0.275" length="0.18" mass="30.28">
+        <origin xyz="0 0 0" rpy="0 0 0" />
+      </xacro:cylinder_inertial>
     </link>
     <link name="${prefix}link_1">
@@ -31,4 +35,7 @@
         <xacro:material_abb_graphite_white/>
       </visual>
+      <xacro:cylinder_inertial radius="0.23" length="0.48" mass="42.41">
+        <origin xyz="0 0 0" rpy="0 0 0" />
+      </xacro:cylinder_inertial>
     </link>
     <link name="${prefix}link_2">
@@ -45,4 +52,7 @@
         <xacro:material_abb_graphite_white/>
       </visual>
+      <xacro:cylinder_inertial radius="0.06" length="1.32" mass="34.32">
+        <origin xyz="0 0 0.65" rpy="0 0 0" />
+      </xacro:cylinder_inertial>
     </link>
     <link name="${prefix}link_3">
@@ -59,4 +69,7 @@
         <xacro:material_abb_graphite_white/>
       </visual>
+      <xacro:cylinder_inertial radius="0.175" length="0.52" mass="51.16">
+        <origin xyz="0 0 0.175" rpy="0 0 0" />
+      </xacro:cylinder_inertial>
     </link>
     <link name="${prefix}link_4">
@@ -73,4 +86,7 @@
         <xacro:material_abb_graphite_white/>
       </visual>
+      <xacro:cylinder_inertial radius="0.08" length="1.03" mass="13.95">
+        <origin xyz="0.8 0 0" rpy="0 ${80} 0" />
+      </xacro:cylinder_inertial>
     </link>
     <link name="${prefix}link_5">
@@ -87,4 +103,7 @@
         <xacro:material_abb_graphite_white/>
       </visual>
+      <xacro:cylinder_inertial radius="0.08" length="0.23" mass="1.5">
+        <origin xyz="0 0 0" rpy="0 0 0" />
+      </xacro:cylinder_inertial>
     </link>
     <link name="${prefix}link_6">
@@ -101,4 +120,7 @@
         <xacro:material_abb_graphite_white/>
       </visual>
+      <xacro:cylinder_inertial radius="0.02" length="0.06" mass="0.27">
+        <origin xyz="0 0 0" rpy="0 0 0" />
+      </xacro:cylinder_inertial>
     </link>
     <!-- end of link list -->

Commit message: add rad unit to expression and fix value

File: robot_specific_config/abb_irb4600_support/urdf/irb4600_40_255_macro.xacro (robot description, xacro)
@@ -90,5 +90,5 @@
       </visual>
       <xacro:cylinder_inertial radius="0.08" length="1.03" mass="13.95">
-        <origin xyz="0.8 0 0" rpy="0 ${80} 0" />
+        <origin xyz="0.8 0 0" rpy="0 ${radians(90)} 0" />
       </xacro:cylinder_inertial>
     </link>
